File: obstacle-avoiding-robo/kicad/obstacle_avoiding_robo/obstacle_avoiding_robo.kicad_sch (KiCad schematic)
At the start: 8 parts, among them J1 Pico 2 W Left Socket P1-P20, J2 Pico 2 W Right Socket P21-P40, J3 TB6612FNG Power/Motor Header, J4 TB6612FNG Logic Header, J5 Left Motor Header, J6 Right Motor Header, J7 3xAA Battery Header, J8 Ultrasonic Sensor Header

Commit message: Added KiCAD designs with gerber files for PCB manufactoring
Parts:
- J3, J4: footprint Connector_PinHeader_2.54mm:PinHeader_1x08_P2.54mm_Vertical -> Connector_PinSocket_2.54mm:PinSocket_1x08_P2.54mm_Vertical
Other:
- note added: "Pico 2 W: 51 x 21 mm, 17.78 mm row spacing; USB at pins 1/40, antenna at pins 20/21."
- note added: "TB6612FNG module: SparkFun ROB-14450, 20.32 mm square, 15.24 mm row spacing."
- note removed: "Pico 2 W is removable: install J1/J2 as 1x20 female socket headers matching the module orientation."
- note removed: "TB6612FNG breakout pin order must match J3/J4 exactly before PCB layout or manufacturing."
Changed lines of the file:
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@@
     (property "Reference" "J3" (at 165.10 38.10 0) (effects (font (size 1.27 1.27))))
     (property "Value" "TB6612FNG Power/Motor Header" (at 165.10 66.04 0) (effects (font (size 1.27 1.27))))
-    (property "Footprint" "Connector_PinHeader_2.54mm:PinHeader_1x08_P2.54mm_Vertical" (at 165.10 50.80 0) (effects (font (size 1.27 1.27)) (hide yes)))
+    (property "Footprint" "Connector_PinSocket_2.54mm:PinSocket_1x08_P2.54mm_Vertical" (at 165.10 50.80 0) (effects (font (size 1.27 1.27)) (hide yes)))
     (property "Datasheet" "" (at 165.10 50.80 0) (effects (font (size 1.27 1.27)) (hide yes)))
     (property "Description" "TB6612FNG Power/Motor Header" (at 165.10 50.80 0) (effects (font (size 1.27 1.27)) (hide yes)))
@@
     (property "Reference" "J4" (at 165.10 71.12 0) (effects (font (size 1.27 1.27))))
     (property "Value" "TB6612FNG Logic Header" (at 165.10 99.06 0) (effects (font (size 1.27 1.27))))
-    (property "Footprint" "Connector_PinHeader_2.54mm:PinHeader_1x08_P2.54mm_Vertical" (at 165.10 83.82 0) (effects (font (size 1.27 1.27)) (hide yes)))
+    (property "Footprint" "Connector_PinSocket_2.54mm:PinSocket_1x08_P2.54mm_Vertical" (at 165.10 83.82 0) (effects (font (size 1.27 1.27)) (hide yes)))
     (property "Datasheet" "" (at 165.10 83.82 0) (effects (font (size 1.27 1.27)) (hide yes)))
     (property "Description" "TB6612FNG Logic Header" (at 165.10 83.82 0) (effects (font (size 1.27 1.27)) (hide yes)))
@@
   (wire (pts (xy 180.34 134.62) (xy 170.18 134.62)) (stroke (width 0) (type solid)))
   (label "GND" (at 170.18 134.62 0) (effects (font (size 1.27 1.27)) (justify left bottom)))
-  (text "Pico 2 W is removable: install J1/J2 as 1x20 female socket headers matching the module orientation." (at 20.32 148.00 0)
+  (text "Pico 2 W: 51 x 21 mm, 17.78 mm row spacing; USB at pins 1/40, antenna at pins 20/21." (at 20.32 148.00 0)
     (effects (font (size 1.27 1.27)) (justify left bottom))
   )
-  (text "TB6612FNG breakout pin order must match J3/J4 exactly before PCB layout or manufacturing." (at 20.32 153.08 0)
+  (text "TB6612FNG module: SparkFun ROB-14450, 20.32 mm square, 15.24 mm row spacing." (at 20.32 153.08 0)
     (effects (font (size 1.27 1.27)) (justify left bottom))
   )
