File: obstacle-avoiding-robo/kicad/obstacle_avoiding_robo/obstacle_avoiding_robo.kicad_pcb (KiCad board)
At the start: 2 copper layers, 80 x 65 mm, 8 parts, among them J1 Pico 2 W Left Socket P1-P20, J2 Pico 2 W Right Socket P21-P40, J3 TB6612FNG Power/Motor Header, J4 TB6612FNG Logic Header, J5 Left Motor Header, J6 Right Motor Header, J7 3xAA Battery Header, J8 Ultrasonic Sensor Header

Commit message: Reposition and route ultrasonic sensor header
Parts:
- moved J8 23.7 mm to (64.2, 36.0), turned to 90 degrees
Routing:
- net /GPIO17_ECHO: track 8.22 -> 37.5 mm
- net /GPIO16_TRIG: track 10.3 -> 37.0 mm
- net /3V3: track 58.4 -> 48.9 mm
Changed lines of the file:
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@@
 	(footprint "Connector_PinHeader_2.54mm:PinHeader_1x04_P2.54mm_Vertical"
 		(layer "F.Cu")
-		(at 50 55)
+		(at 64.2 36 90)
 		(descr "Through hole straight pin header, 1x04, 2.54mm pitch, single row")
 		(tags "Through hole pin header THT 1x04 2.54mm single row")
 		(property "Reference" "J8"
-			(at 0 -2.38 0)
+			(at 0 -2.38 90)
 			(layer "F.SilkS")
 			(effects
@@
 		)
 		(property "Value" "Ultrasonic Sensor Header"
-			(at 0 10 0)
+			(at 0 10 90)
 			(layer "F.Fab")
 			(effects
@@
 		)
 		(property "Datasheet" ""
-			(at 0 0 0)
+			(at 0 0 90)
 			(layer "F.Fab")
 			(hide yes)
@@
 		)
 		(property "Description" "Ultrasonic Sensor Header"
-			(at 0 0 0)
+			(at 0 0 90)
 			(layer "F.Fab")
 			(hide yes)
@@
 		)
 		(property "KiLib_Generator" "connector/pin_header_socket"
-			(at 0 0 0)
+			(at 0 0 90)
 			(layer "F.SilkS")
 			(hide yes)
@@
 		)
 		(fp_line
+			(start 1.38 1.27)
+			(end 1.38 9)
+			(stroke
+				(width 0.12)
+				(type solid)
+			)
+			(layer "F.SilkS")
+		)
+		(fp_line
+			(start -1.38 1.27)
+			(end 1.38 1.27)
+			(stroke
+				(width 0.12)
+				(type solid)
+			)
+			(layer "F.SilkS")
+		)
+		(fp_line
 			(start -1.38 1.27)
 			(end -1.38 9)
@@
 		)
 		(fp_line
-			(start -1.38 1.27)
-			(end 1.38 1.27)
-			(stroke
-				(width 0.12)
-				(type solid)
-			)
-			(layer "F.SilkS")
-		)
-		(fp_line
 			(start -1.38 9)
-			(end 1.38 9)
-			(stroke
-				(width 0.12)
-				(type solid)
-			)
-			(layer "F.SilkS")
-		)
-		(fp_line
-			(start 1.38 1.27)
 			(end 1.38 9)
 			(stroke
@@
 		)
 		(fp_line
+			(start 1.27 -1.27)
+			(end 1.27 8.89)
+			(stroke
+				(width 0.1)
+				(type solid)
+			)
+			(layer "F.Fab")
+		)
+		(fp_line
+			(start -0.635 -1.27)
+			(end 1.27 -1.27)
+			(stroke
+				(width 0.1)
+				(type solid)
+			)
+			(layer "F.Fab")
+		)
+		(fp_line
 			(start -1.27 -0.635)
 			(end -0.635 -1.27)
@@
 		)
 		(fp_line
+			(start 1.27 8.89)
+			(end -1.27 8.89)
+			(stroke
+				(width 0.1)
+				(type solid)
+			)
+			(layer "F.Fab")
+		)
+		(fp_line
 			(start -1.27 8.89)
 			(end -1.27 -0.635)
@@
 			(layer "F.Fab")
 		)
-		(fp_line
-			(start -0.635 -1.27)
-			(end 1.27 -1.27)
-			(stroke
-				(width 0.1)
-				(type solid)
-			)
-			(layer "F.Fab")
-		)
-		(fp_line
-			(start 1.27 -1.27)
-			(end 1.27 8.89)
-			(stroke
-				(width 0.1)
-				(type solid)
-			)
-			(layer "F.Fab")
-		)
-		(fp_line
-			(start 1.27 8.89)
-			(end -1.27 8.89)
-			(stroke
-				(width 0.1)
-				(type solid)
-			)
-			(layer "F.Fab")
-		)
 		(fp_text user "${REFERENCE}"
-			(at 0 3.81 90)
+			(at 0 3.81 0)
 			(layer "F.Fab")
 			(effects
@@
 		)
 		(pad "1" thru_hole rect
-			(at 0 0)
+			(at 0 0 90)
 			(size 1.7 1.7)
 			(drill 1)
@@
 		)
 		(pad "2" thru_hole circle
-			(at 0 2.54)
+			(at 0 2.54 90)
 			(size 1.7 1.7)
 			(drill 1)
@@
 		)
 		(pad "3" thru_hole circle
-			(at 0 5.08)
+			(at 0 5.08 90)
 			(size 1.7 1.7)
 			(drill 1)
@@
 		)
 		(pad "4" thru_hole circle
-			(at 0 7.62)
+			(at 0 7.62 90)
 			(size 1.7 1.7)
 			(drill 1)
@@
 		)
 	)
-	(gr_text "VCC"
-		(at 46.2 55 0)
-		(layer "F.SilkS")
-		(effects
-			(font
-				(size 0.8 0.8)
-				(thickness 0.12)
-			)
-		)
-	)
-	(gr_text "TRIG"
-		(at 46.2 57.54 0)
-		(layer "F.SilkS")
-		(effects
-			(font
-				(size 0.8 0.8)
-				(thickness 0.12)
-			)
-		)
-	)
-	(gr_text "ECHO"
-		(at 46.2 60.08 0)
-		(layer "F.SilkS")
-		(effects
-			(font
-				(size 0.8 0.8)
-				(thickness 0.12)
-			)
-		)
-	)
-	(gr_text "GND"
-		(at 46.2 62.62 0)
-		(layer "F.SilkS")
-		(effects
-			(font
-				(size 0.8 0.8)
-				(thickness 0.12)
-			)
-		)
-	)
-	(gr_text "ULTRASONIC"
-		(at 56 52.2 0)
-		(layer "F.SilkS")
-		(effects
-			(font
-				(size 0.8 0.8)
-				(thickness 0.12)
-			)
-		)
-	)
 	(gr_text "TB6612FNG ROB-14450"
 		(at 58.12 25.7 0)
@@
 		)
 	)
+	(gr_text "VCC"
+		(at 64.2 39 0)
+		(layer "F.SilkS")
+		(effects
+			(font
+				(size 0.8 0.8)
+				(thickness 0.12)
+			)
+		)
+	)
+	(gr_text "TRIG"
+		(at 66.74 40 0)
+		(layer "F.SilkS")
+		(effects
+			(font
+				(size 0.8 0.8)
+				(thickness 0.12)
+			)
+		)
+	)
+	(gr_text "ULTRASONIC"
+		(at 68 42 0)
+		(layer "F.SilkS")
+		(effects
+			(font
+				(size 0.8 0.8)
+				(thickness 0.12)
+			)
+		)
+	)
+	(gr_text "ECHO"
+		(at 69.28 39 0)
+		(layer "F.SilkS")
+		(effects
+			(font
+				(size 0.8 0.8)
+				(thickness 0.12)
+			)
+		)
+	)
 	(gr_text "GND"
 		(at 70 3.27 0)
@@
 	(gr_text "+"
 		(at 70.5 25 0)
+		(layer "F.SilkS")
+		(effects
+			(font
+				(size 0.8 0.8)
+				(thickness 0.12)
+			)
+		)
+	)
+	(gr_text "GND"
+		(at 71.82 40 0)
 		(layer "F.SilkS")
 		(effects
@@
 	)
 	(segment
-		(start 44.91 62.63)
-		(end 50 57.54)
-		(width 0.25)
-		(layer "B.Cu")
+		(start 41.78 62.63)
+		(end 66.74 37.67)
+		(width 0.25)
+		(layer "F.Cu")
 		(net "/GPIO16_TRIG")
 	)
 	(segment
-		(start 41.78 62.63)
-		(end 44.91 62.63)
-		(width 0.25)
-		(layer "B.Cu")
+		(start 66.74 37.67)
+		(end 66.74 36)
+		(width 0.25)
+		(layer "F.Cu")
 		(net "/GPIO16_TRIG")
 	)
 	(segment
-		(start 49.99 60.09)
-		(end 50 60.08)
-		(width 0.25)
-		(layer "F.Cu")
+		(start 45.19 60.09)
+		(end 69.28 36)
+		(width 0.25)
+		(layer "B.Cu")
 		(net "/GPIO17_ECHO")
 	)
 	(segment
 		(start 41.78 60.09)
-		(end 49.99 60.09)
-		(width 0.25)
-		(layer "F.Cu")
+		(end 45.19 60.09)
+		(width 0.25)
+		(layer "B.Cu")
 		(net "/GPIO17_ECHO")
 	)
@@
 	)
 	(segment
-		(start 50 55)
-		(end 50 28.03)
+		(start 64.2 36)
+		(end 57.97 36)
 		(width 0.8)
 		(layer "F.Cu")
@@
 	)
 	(segment
-		(start 50 28.03)
-		(end 46.5 24.53)
-		(width 0.8)
-		(layer "F.Cu")
-		(net "/3V3")
-	)
-	(segment
 		(start 65.739999 18.51)
 		(end 59.47 18.51)
 		(width 0.8)
 		(layer "F.Cu")
+		(net "/3V3")
+	)
+	(segment
+		(start 57.97 36)
+		(end 46.5 24.53)
+		(width 0.8)
+		(layer "F.Cu")
